Commit message: congig Rviz2 + moveit2

File: install/Robot_description/share/Robot_description/urdf/Robot.xacro (robot description, xacro)
@@ -189,5 +189,5 @@
   <child link="link1_1"/>
   <axis xyz="-0.000105 6.8e-05 1.0"/>
-  <limit upper="3.1415927" lower="-3.1415927" effort="100" velocity="100"/>
+  <limit upper="3.1415927" lower="-3.1415927" effort="100" velocity="100.0"/>
 </joint>
 <joint name="Joint2" type="revolute">
@@ -196,5 +196,5 @@
   <child link="link2_1"/>
   <axis xyz="0 1 0"/>
-  <limit upper="1.919862" lower="-1.919862" effort="100" velocity="100"/>
+  <limit upper="1.919862" lower="-1.919862" effort="100" velocity="100.0"/>
 </joint>
 <joint name="Joint3" type="revolute">
@@ -203,5 +203,5 @@
   <child link="link3_1"/>
   <axis xyz="0 1 0"/>
-  <limit upper="2.10" lower="-2.10" effort="100" velocity="100"/>
+  <limit upper="2.10" lower="-2.10" effort="100" velocity="100.0"/>
 </joint>
 <joint name="Joint4" type="revolute">
@@ -210,5 +210,5 @@
   <child link="link4_1"/>
   <axis xyz="0 0 1"/>
-  <limit upper="3.1415927" lower="-3.1415927" effort="100" velocity="100"/>
+  <limit upper="3.1415927" lower="-3.1415927" effort="100" velocity="100.0"/>
 </joint>
 <joint name="Joint5" type="revolute">
@@ -217,5 +217,5 @@
   <child link="link5_1"/>
   <axis xyz="0 1 0"/>
-  <limit upper="1.832596" lower="-1.832596" effort="100" velocity="100"/>
+  <limit upper="1.832596" lower="-1.832596" effort="100" velocity="100.0"/>
 </joint>
 <joint name="Joint6" type="revolute">
@@ -224,5 +224,5 @@
   <child link="link6_1"/>
   <axis xyz="0 0 1"/>
-  <limit upper="3.1415927" lower="-3.1415927" effort="100" velocity="100"/>
+  <limit upper="3.1415927" lower="-3.1415927" effort="100" velocity="100.0"/>
 </joint>
 <joint name="Servo Joint" type="revolute">
@@ -231,5 +231,5 @@
   <child link="Servo_Gear_1"/>
   <axis xyz="0 0 -1"/>
-  <limit upper="0.959931" lower="0.523599" effort="100" velocity="100"/>
+  <limit upper="0.959931" lower="0.523599" effort="100" velocity="100.0"/>
 </joint>
 <joint name="Idol Joint" type="revolute">
@@ -238,5 +238,5 @@
   <child link="Idol_Gear_1"/>
   <axis xyz="0 0 1"/>
-  <limit upper="0.959931" lower="0.523599" effort="100" velocity="100"/>
+  <limit upper="0.959931" lower="0.523599" effort="100" velocity="100.0"/>
 </joint>
 </robot>

File: install/robot_moveit_config/share/robot_moveit_config/config/Robot.ros2_control.xacro (robot description, xacro)
@@ -10,4 +10,5 @@
             <joint name="Joint1">
                 <command_interface name="position"/>
+                <command_interface name="velocity"/>
                 <state_interface name="position">
                   <param name="initial_value">${initial_positions['Joint1']}</param>
@@ -17,4 +18,5 @@
             <joint name="Joint2">
                 <command_interface name="position"/>
+                <command_interface name="velocity"/>
                 <state_interface name="position">
                   <param name="initial_value">${initial_positions['Joint2']}</param>
@@ -24,4 +26,5 @@
             <joint name="Joint3">
                 <command_interface name="position"/>
+                <command_interface name="velocity"/>
                 <state_interface name="position">
                   <param name="initial_value">${initial_positions['Joint3']}</param>
@@ -31,4 +34,5 @@
             <joint name="Joint4">
                 <command_interface name="position"/>
+                <command_interface name="velocity"/>
                 <state_interface name="position">
                   <param name="initial_value">${initial_positions['Joint4']}</param>
@@ -38,4 +42,5 @@
             <joint name="Joint5">
                 <command_interface name="position"/>
+                <command_interface name="velocity"/>
                 <state_interface name="position">
                   <param name="initial_value">${initial_positions['Joint5']}</param>
@@ -45,4 +50,5 @@
             <joint name="Joint6">
                 <command_interface name="position"/>
+                <command_interface name="velocity"/>
                 <state_interface name="position">
                   <param name="initial_value">${initial_positions['Joint6']}</param>
@@ -52,4 +58,5 @@
             <joint name="Idol Joint">
                 <command_interface name="position"/>
+                <command_interface name="velocity"/>
                 <state_interface name="position">
                   <param name="initial_value">${initial_positions['Idol Joint']}</param>
@@ -59,4 +66,5 @@
             <joint name="Servo Joint">
                 <command_interface name="position"/>
+                <command_interface name="velocity"/>
                 <state_interface name="position">
                   <param name="initial_value">${initial_positions['Servo Joint']}</param>

File: install/robot_moveit_config/share/robot_moveit_config/config/Robot.urdf.xacro (robot description, xacro)
@@ -3,311 +3,7 @@
     <xacro:arg name="initial_positions_file" default="initial_positions.yaml" />
     <!-- Import Robot urdf file -->
-    <!-- xacro:include filename="/home/julien/Documents/ros/robot_arm/src/Robot_description/urdf/Robot.xacro" /-->
-    <xacro:include filename="/home/julien/Documents/ros/robot_arm/src/Robot_description/urdf/materials.xacro" />
-    <xacro:include filename="/home/julien/Documents/ros/robot_arm/src/Robot_description/urdf/Robot.trans" />
-    <xacro:include filename="/home/julien/Documents/ros/robot_arm/src/Robot_description/urdf/Robot.gazebo" />
-    <link name="base_link">
-    <inertial>
-        <origin xyz="9.323197461062662e-06 -2.179181289320399e-06 0.03766434672102797" rpy="0 0 0"/>
-        <mass value="0.6555115079798821"/>
-        <inertia ixx="0.001559" iyy="0.001558" izz="0.002695" ixy="-0.0" iyz="0.0" ixz="-0.0"/>
-    </inertial>
-    <visual>
-        <origin xyz="0 0 0" rpy="0 0 0"/>
-        <geometry>
-        <mesh filename="package://Robot_description/meshes/base_link.stl" scale="0.001 0.001 0.001"/>
-        </geometry>
-        <material name="silver"/>
-    </visual>
-    <collision>
-        <origin xyz="0 0 0" rpy="0 0 0"/>
-        <geometry>
-        <mesh filename="package://Robot_description/meshes/base_link.stl" scale="0.001 0.001 0.001"/>
-        </geometry>
-    </collision>
-    </link>
-    <link name="link1_1">
-    <inertial>
-        <origin xyz="-8.747364957463794e-05 0.00023000695233989162 0.08027934823103827" rpy="0 0 0"/>
-        <mass value="1.9598700732514862"/>
-        <inertia ixx="0.009232" iyy="0.013036" izz="0.008743" ixy="-0.000121" iyz="-2e-06" ixz="-9e-06"/>
-    </inertial>
-    <visual>
-        <origin xyz="0 0 0" rpy="0 0 0"/>
-        <geometry>
-        <mesh filename="package://Robot_description/meshes/link1_1.stl" scale="0.001 0.001 0.001"/>
-        </geometry>
-        <material name="silver"/>
-    </visual>
-    <collision>
-        <origin xyz="0 0 0" rpy="0 0 0"/>
-        <geometry>
-        <mesh filename="package://Robot_description/meshes/link1_1.stl" scale="0.001 0.001 0.001"/>
-        </geometry>
-    </collision>
-    </link>
-    <link name="link2_1">
-    <inertial>
-        <origin xyz="-0.03550849992822761 -0.20005697525257984 0.10074520526952119" rpy="0 0 0"/>
-        <mass value="1.9144645074140343"/>
-        <inertia ixx="0.015946" iyy="0.016692" izz="0.003538" ixy="-2.5e-05" iyz="0.000266" ixz="-0.000131"/>
-    </inertial>
-    <visual>
-        <origin xyz="0 0 0" rpy="0 0 0"/>
-        <geometry>
-        <mesh filename="package://Robot_description/meshes/link2_1.stl" scale="0.001 0.001 0.001"/>
-        </geometry>
-        <material name="silver"/>
-    </visual>
-    <collision>
-        <origin xyz="0 0 0" rpy="0 0 0"/>
-        <geometry>
-        <mesh filename="package://Robot_description/meshes/link2_1.stl" scale="0.001 0.001 0.001"/>
-        </geometry>
-    </collision>
-    </link>
-    <link name="link3_1">
-    <inertial>
-        <origin xyz="-0.002261294975221836 -0.06191695522524358 0.5730413856217828" rpy="0 0 0"/>
-        <mass value="0.7274515218419347"/>
-        <inertia ixx="0.002081" iyy="0.001928" izz="0.000789" ixy="7e-06" iyz="0.000373" ixz="-1.9e-05"/>
-    </inertial>
-    <visual>
-        <origin xyz="0 0 0" rpy="0 0 0"/>
-        <geometry>
-        <mesh filename="package://Robot_description/meshes/link3_1.stl" scale="0.001 0.001 0.001"/>
-        </geometry>
-        <material name="silver"/>
-    </visual>
-    <collision>
-        <origin xyz="0 0 0" rpy="0 0 0"/>
-        <geometry>
-        <mesh filename="package://Robot_description/meshes/link3_1.stl" scale="0.001 0.001 0.001"/>
-        </geometry>
-    </collision>
-    </link>
-    <link name="link4_1">
-    <inertial>
-        <origin xyz="0.08399775381594644 -0.46346924906243314 0.0999798189364719" rpy="0 0 0"/>
-        <mass value="0.32455418653717066"/>
-        <inertia ixx="0.000669" iyy="0.000571" izz="0.000352" ixy="4.1e-05" iyz="6.1e-05" ixz="7e-06"/>
-    </inertial>
-    <visual>
-        <origin xyz="0 0 0" rpy="0 0 0"/>
-        <geometry>
-        <mesh filename="package://Robot_description/meshes/link4_1.stl" scale="0.001 0.001 0.001"/>
-        </geometry>
-        <material name="silver"/>
-    </visual>
-    <collision>
-        <origin xyz="0 0 0" rpy="0 0 0"/>
-        <geometry>
-        <mesh filename="package://Robot_description/meshes/link4_1.stl" scale="0.001 0.001 0.001"/>
-        </geometry>
-    </collision>
-    </link>
-    <link name="link5_1">
-    <inertial>
-        <origin xyz="-0.18454465996686803 0.41770479167069396 0.21286940543338817" rpy="0 0 0"/>
-        <mass value="0.1607410659493192"/>
-        <inertia ixx="9.1e-05" iyy="0.000104" izz="7.9e-05" ixy="-5e-06" iyz="5e-06" ixz="-8e-06"/>
-    </inertial>
-    <visual>
-        <origin xyz="0 0 0" rpy="0 0 0"/>
-        <geometry>
-        <mesh filename="package://Robot_description/meshes/link5_1.stl" scale="0.001 0.001 0.001"/>
-        </geometry>
-        <material name="silver"/>
-    </visual>
-    <collision>
-        <origin xyz="0 0 0" rpy="0 0 0"/>
-        <geometry>
-        <mesh filename="package://Robot_description/meshes/link5_1.stl" scale="0.001 0.001 0.001"/>
-        </geometry>
-    </collision>
-    </link>
-    <link name="link6_1">
-    <inertial>
-        <origin xyz="-0.1139190355815723 0.43442970533659214 0.38100115968800496" rpy="0 0 0"/>
-        <mass value="0.01865052429923146"/>
-        <inertia ixx="1e-05" iyy="6e-06" izz="1e-05" ixy="2e-06" iyz="-1e-06" ixz="-1e-06"/>
-    </inertial>
-    <visual>
-        <origin xyz="0 0 0" rpy="0 0 0"/>
-        <geometry>
-        <mesh filename="package://Robot_description/meshes/link6_1.stl" scale="0.001 0.001 0.001"/>
-        </geometry>
-        <material name="silver"/>
-    </visual>
-    <collision>
-        <origin xyz="0 0 0" rpy="0 0 0"/>
-        <geometry>
-        <mesh filename="package://Robot_description/meshes/link6_1.stl" scale="0.001 0.001 0.001"/>
-        </geometry>
-    </collision>
-    </link>
-    <link name="Servo_Gear_1">
-    <inertial>
-        <origin xyz="0.018998787739794347 -0.03233241707548999 0.024569258659072113" rpy="0 0 0"/>
-        <mass value="0.015458635829547249"/>
-        <inertia ixx="1.4e-05" iyy="1e-05" izz="9e-06" ixy="3e-06" iyz="6e-06" ixz="-4e-06"/>
-    </inertial>
-    <visual>
-        <origin xyz="0 0 0" rpy="0 0 0"/>
-        <geometry>
-        <mesh filename="package://Robot_description/meshes/Servo_Gear_1.stl" scale="0.001 0.001 0.001"/>
-        </geometry>
-        <material name="silver"/>
-    </visual>
-    <collision>
-        <origin xyz="0 0 0" rpy="0 0 0"/>
-        <geometry>
-        <mesh filename="package://Robot_description/meshes/Servo_Gear_1.stl" scale="0.001 0.001 0.001"/>
-        </geometry>
-    </collision>
-    </link>
-    <link name="Idol_Gear_1">
-    <inertial>
-        <origin xyz="0.01859007116218464 0.005649685131553797 0.04057153069940722" rpy="0 0 0"/>
-        <mass value="0.01558102330322005"/>
-        <inertia ixx="1.4e-05" iyy="1.6e-05" izz="3e-06" ixy="0.0" iyz="0.0" ixz="-5e-06"/>
-    </inertial>
-    <visual>
-        <origin xyz="0 0 0" rpy="0 0 0"/>
-        <geometry>
-        <mesh filename="package://Robot_description/meshes/Idol_Gear_1.stl" scale="0.001 0.001 0.001"/>
-        </geometry>
-        <material name="silver"/>
-    </visual>
-    <collision>
-        <origin xyz="0 0 0" rpy="0 0 0"/>
-        <geometry>
-        <mesh filename="package://Robot_description/meshes/Idol_Gear_1.stl" scale="0.001 0.001 0.001"/>
-        </geometry>
-    </collision>
-    </link>
-    <joint name="Joint1" type="revolute">
-    <origin xyz="-7e-06 4e-06 0.065" rpy="0 0 0"/>
-    <parent link="base_link"/>
-    <child link="link1_1"/>
-    <axis xyz="-0.000105 6.8e-05 1.0"/>
-    <limit upper="3.1415927" lower="-3.1415927" effort="100" velocity="100"/>
-    </joint>
-    <joint name="Joint2" type="revolute">
-    <origin xyz="0 0 0.1655" rpy="0 0 0"/>
-    <parent link="link1_1"/>
-    <child link="link2_1"/>
-    <axis xyz="0 1 0"/>
-    <limit upper="1.919862" lower="-1.919862" effort="100" velocity="100"/>
-    </joint>
-    <joint name="Joint3" type="revolute">
-    <origin xyz="0.0025 0 0.222" rpy="0 0 0"/>
-    <parent link="link2_1"/>
-    <child link="link3_1"/>
-    <axis xyz="0 1 0"/>
-    <limit upper="2.10" lower="-2.10" effort="100" velocity="100"/>
-    </joint>
-    <joint name="Joint4" type="revolute">
-    <origin xyz="0 0 0.1291" rpy="0 0 0"/>
-    <parent link="link3_1"/>
-    <child link="link4_1"/>
-    <axis xyz="0 0 1"/>
-    <limit upper="3.1415927" lower="-3.1415927" effort="100" velocity="100"/>
-    </joint>
-    <joint name="Joint5" type="revolute">
-    <origin xyz="0 0 0.095" rpy="0 0 0"/>
-    <parent link="link4_1"/>
-    <child link="link5_1"/>
-    <axis xyz="0 1 0"/>
-    <limit upper="1.832596" lower="-1.832596" effort="100" velocity="100"/>
-    </joint>
-    <joint name="Joint6" type="revolute">
-    <origin xyz="0 0 0.0469" rpy="0 0 0"/>
-    <parent link="link5_1"/>
-    <child link="link6_1"/>
-    <axis xyz="0 0 1"/>
-    <limit upper="3.1415927" lower="-3.1415927" effort="100" velocity="100"/>
-    </joint>
-    <joint name="Servo Joint" type="revolute">
-    <origin xyz="0 -0.014 0.024" rpy="0 -1.5708 0"/>
-    <parent link="link6_1"/>
-    <child link="Servo_Gear_1"/>
-    <axis xyz="0 0 -1"/>
-    <limit upper="0.959931" lower="0.523599" effort="100" velocity="100"/>
-    </joint>
-    <joint name="Idol Joint" type="revolute">
-    <origin xyz="0 0.014 0.024" rpy="0 -1.5708 0"/>
-    <parent link="link6_1"/>
-    <child link="Idol_Gear_1"/>
-    <axis xyz="0 0 1"/>
-    <limit upper="0.959931" lower="0.523599" effort="100" velocity="100"/>
-    </joint>
+    <xacro:include filename="$(find Robot_description)/urdf/Robot.xacro" />
     <!-- Import control_xacro -->
-    <!--xacro:include filename="Robot.ros2_control.xacro" /-->
-    <xacro:macro name="Robot_ros2_control" params="name initial_positions_file">
-        <xacro:property name="initial_positions" value="${load_yaml(initial_positions_file)['initial_positions']}"/>
-        <ros2_control name="${name}" type="system">
-            <hardware>
-                <!-- By default, set up controllers for simulation. This won't work on real hardware -->
-                <plugin>mock_components/GenericSystem</plugin>
-            </hardware>
-            <joint name="Joint1">
-                <command_interface name="position"/>
-                <state_interface name="position">
-                  <param name="initial_value">${initial_positions['Joint1']}</param>
-                </state_interface>
-                <state_interface name="velocity"/>
-            </joint>
-            <joint name="Joint2">
-                <command_interface name="position"/>
-                <state_interface name="position">
-                  <param name="initial_value">${initial_positions['Joint2']}</param>
-                </state_interface>
-                <state_interface name="velocity"/>
-            </joint>
-            <joint name="Joint3">
-                <command_interface name="position"/>
-                <state_interface name="position">
-                  <param name="initial_value">${initial_positions['Joint3']}</param>
-                </state_interface>
-                <state_interface name="velocity"/>
-            </joint>
-            <joint name="Joint4">
-                <command_interface name="position"/>
-                <state_interface name="position">
-                  <param name="initial_value">${initial_positions['Joint4']}</param>
-                </state_interface>
-                <state_interface name="velocity"/>
-            </joint>
-            <joint name="Joint5">
-                <command_interface name="position"/>
-                <state_interface name="position">
-                  <param name="initial_value">${initial_positions['Joint5']}</param>
-                </state_interface>
-                <state_interface name="velocity"/>
-            </joint>
-            <joint name="Joint6">
-                <command_interface name="position"/>
-                <state_interface name="position">
-                  <param name="initial_value">${initial_positions['Joint6']}</param>
-                </state_interface>
-                <state_interface name="velocity"/>
-            </joint>
-            <joint name="Idol Joint">
-                <command_interface name="position"/>
-                <state_interface name="position">
-                  <param name="initial_value">${initial_positions['Idol Joint']}</param>
-                </state_interface>
-                <state_interface name="velocity"/>
-            </joint>
-            <joint name="Servo Joint">
-                <command_interface name="position"/>
-                <state_interface name="position">
-                  <param name="initial_value">${initial_positions['Servo Joint']}</param>
-                </state_interface>
-                <state_interface name="velocity"/>
-            </joint>
-        </ros2_control>
-    </xacro:macro>
+    <xacro:include filename="Robot.ros2_control.xacro" />
     <xacro:Robot_ros2_control name="FakeSystem" initial_positions_file="$(arg initial_positions_file)"/>
 </robot>

Commit message: Ajout de la kinematics

File: install/Robot_description/share/Robot_description/urdf/Robot.xacro (robot description, xacro)
@@ -189,5 +189,5 @@
   <child link="link1_1"/>
   <axis xyz="-0.000105 6.8e-05 1.0"/>
-  <limit upper="3.1415927" lower="-3.1415927" effort="100" velocity="100.0"/>
+  <limit upper="1.95" lower="-1.95" effort="100" velocity="100.0"/>
 </joint>
 <joint name="Joint2" type="revolute">
@@ -196,5 +196,5 @@
   <child link="link2_1"/>
   <axis xyz="0 1 0"/>
-  <limit upper="1.919862" lower="-1.919862" effort="100" velocity="100.0"/>
+  <limit upper="1.92" lower="-1.5" effort="100" velocity="100.0"/>
 </joint>
 <joint name="Joint3" type="revolute">
@@ -217,5 +217,5 @@
   <child link="link5_1"/>
   <axis xyz="0 1 0"/>
-  <limit upper="1.832596" lower="-1.832596" effort="100" velocity="100.0"/>
+  <limit upper="1.7" lower="-1.7" effort="100" velocity="100.0"/>
 </joint>
 <joint name="Joint6" type="revolute">
@@ -231,5 +231,5 @@
   <child link="Servo_Gear_1"/>
   <axis xyz="0 0 -1"/>
-  <limit upper="0.959931" lower="0.523599" effort="100" velocity="100.0"/>
+  <limit upper="2.28" lower="0.523599" effort="100" velocity="100.0"/>
 </joint>
 <joint name="Idol Joint" type="revolute">
@@ -238,5 +238,5 @@
   <child link="Idol_Gear_1"/>
   <axis xyz="0 0 1"/>
-  <limit upper="0.959931" lower="0.523599" effort="100" velocity="100.0"/>
+  <limit upper="2.28" lower="0.523599" effort="100" velocity="100.0"/>
 </joint>
 </robot>
