Commit message: MAJ move_cpp

File: ros2_ws_robot/install/robot_description/share/robot_description/urdf/Robot.xacro (robot description, xacro)
@@ -239,4 +239,5 @@
   <axis xyz="0 0 -1"/>
   <limit upper="0" lower="-1.5708" effort="100" velocity="100.0"/>
+  <mimic joint="Servo Joint"/>
 </joint>
 </robot>

File: ros2_ws_robot/install/robot_moveit_config/share/robot_moveit_config/config/Robot.ros2_control.xacro (robot description, xacro)
@@ -13,4 +13,5 @@
                   <param name="initial_value">${initial_positions['Joint1']}</param>
                 </state_interface>
+                <state_interface name="velocity"/>
             </joint>
             <joint name="Joint2">
@@ -19,4 +20,5 @@
                   <param name="initial_value">${initial_positions['Joint2']}</param>
                 </state_interface>
+                <state_interface name="velocity"/>
             </joint>
             <joint name="Joint3">
@@ -25,4 +27,5 @@
                   <param name="initial_value">${initial_positions['Joint3']}</param>
                 </state_interface>
+                <state_interface name="velocity"/>
             </joint>
             <joint name="Joint4">
@@ -31,4 +34,5 @@
                   <param name="initial_value">${initial_positions['Joint4']}</param>
                 </state_interface>
+                <state_interface name="velocity"/>
             </joint>
             <joint name="Joint5">
@@ -37,4 +41,5 @@
                   <param name="initial_value">${initial_positions['Joint5']}</param>
                 </state_interface>
+                <state_interface name="velocity"/>
             </joint>
             <joint name="Joint6">
@@ -43,10 +48,5 @@
                   <param name="initial_value">${initial_positions['Joint6']}</param>
                 </state_interface>
-            </joint>
-            <joint name="Idol Joint">
-                <command_interface name="position"/>
-                <state_interface name="position">
-                  <param name="initial_value">${initial_positions['Idol Joint']}</param>
-                </state_interface>
+                <state_interface name="velocity"/>
             </joint>
             <joint name="Servo Joint">
@@ -55,4 +55,5 @@
                   <param name="initial_value">${initial_positions['Servo Joint']}</param>
                 </state_interface>
+                <state_interface name="velocity"/>
             </joint>
         </ros2_control>

Commit message: Développement TicTacToe

File: ros2_ws_robot/install/robot_description/share/robot_description/urdf/Robot.xacro (robot description, xacro)
@@ -5,9 +5,9 @@
 <xacro:include filename="Robot.gazebo" />
 <link name="base_link">
-  <inertial>
+  <!-- <inertial>
     <origin xyz="9.323197461062662e-06 -2.179181289320399e-06 0.03766434672102797" rpy="0 0 0"/>
     <mass value="0.6555115079798821"/>
     <inertia ixx="0.001559" iyy="0.001558" izz="0.002695" ixy="-0.0" iyz="0.0" ixz="-0.0"/>
-  </inertial>
+  </inertial> -->
   <visual>
     <origin xyz="0 0 0" rpy="0 0 0"/>
@@ -196,5 +196,5 @@
   <child link="link2_1"/>
   <axis xyz="0 1 0"/>
-  <limit upper="1.92" lower="-1.5" effort="100" velocity="100.0"/>
+  <limit upper="1.92" lower="-0.873" effort="100" velocity="100.0"/>
 </joint>
 <joint name="Joint3" type="revolute">
@@ -210,5 +210,5 @@
   <child link="link4_1"/>
   <axis xyz="0 0 1"/>
-  <limit upper="3.1415927" lower="-3.1415927" effort="100" velocity="100.0"/>
+  <limit upper="2.36" lower="-2.36" effort="100" velocity="100.0"/>
 </joint>
 <joint name="Joint5" type="revolute">
@@ -224,5 +224,5 @@
   <child link="link6_1"/>
   <axis xyz="0 0 1"/>
-  <limit upper="3.1415927" lower="-3.1415927" effort="100" velocity="100.0"/>
+  <limit upper="2.36" lower="-2.36" effort="100" velocity="100.0"/>
 </joint>
 <joint name="Servo Joint" type="revolute">
@@ -237,7 +237,7 @@
   <parent link="link6_1"/>
   <child link="Idol_Gear_1"/>
+  <mimic joint="Servo Joint"/>
   <axis xyz="0 0 -1"/>
   <limit upper="0" lower="-1.5708" effort="100" velocity="100.0"/>
-  <mimic joint="Servo Joint"/>
 </joint>
 </robot>

Commit message: 18_09_15h49

File: ros2_ws_robot/install/robot_description/share/robot_description/urdf/Robot.xacro (robot description, xacro)
@@ -189,5 +189,5 @@
   <child link="link1_1"/>
   <axis xyz="-0.000105 6.8e-05 1.0"/>
-  <limit upper="1.95" lower="-1.95" effort="100" velocity="100.0"/>
+  <limit upper="1.658" lower="-1.658" effort="100" velocity="100.0"/>
 </joint>
 <joint name="Joint2" type="revolute">

Commit message: 18_09_19h51

File: ros2_ws_robot/install/robot_description/share/robot_description/urdf/Robot.xacro (robot description, xacro)
@@ -5,9 +5,4 @@
 <xacro:include filename="Robot.gazebo" />
 <link name="base_link">
-  <!-- <inertial>
-    <origin xyz="9.323197461062662e-06 -2.179181289320399e-06 0.03766434672102797" rpy="0 0 0"/>
-    <mass value="0.6555115079798821"/>
-    <inertia ixx="0.001559" iyy="0.001558" izz="0.002695" ixy="-0.0" iyz="0.0" ixz="-0.0"/>
-  </inertial> -->
   <visual>
     <origin xyz="0 0 0" rpy="0 0 0"/>
@@ -25,9 +20,4 @@
 </link>
 <link name="link1_1">
-  <inertial>
-    <origin xyz="-8.747364957463794e-05 0.00023000695233989162 0.08027934823103827" rpy="0 0 0"/>
-    <mass value="1.9598700732514862"/>
-    <inertia ixx="0.009232" iyy="0.013036" izz="0.008743" ixy="-0.000121" iyz="-2e-06" ixz="-9e-06"/>
-  </inertial>
   <visual>
     <origin xyz="0 0 0" rpy="0 0 0"/>
@@ -45,9 +35,4 @@
 </link>
 <link name="link2_1">
-  <inertial>
-    <origin xyz="-0.03550849992822761 -0.20005697525257984 0.10074520526952119" rpy="0 0 0"/>
-    <mass value="1.9144645074140343"/>
-    <inertia ixx="0.015946" iyy="0.016692" izz="0.003538" ixy="-2.5e-05" iyz="0.000266" ixz="-0.000131"/>
-  </inertial>
   <visual>
     <origin xyz="0 0 0" rpy="0 0 0"/>
@@ -65,9 +50,4 @@
 </link>
 <link name="link3_1">
-  <inertial>
-    <origin xyz="-0.002261294975221836 -0.06191695522524358 0.5730413856217828" rpy="0 0 0"/>
-    <mass value="0.7274515218419347"/>
-    <inertia ixx="0.002081" iyy="0.001928" izz="0.000789" ixy="7e-06" iyz="0.000373" ixz="-1.9e-05"/>
-  </inertial>
   <visual>
     <origin xyz="0 0 0" rpy="0 0 0"/>
@@ -85,9 +65,4 @@
 </link>
 <link name="link4_1">
-  <inertial>
-    <origin xyz="0.08399775381594644 -0.46346924906243314 0.0999798189364719" rpy="0 0 0"/>
-    <mass value="0.32455418653717066"/>
-    <inertia ixx="0.000669" iyy="0.000571" izz="0.000352" ixy="4.1e-05" iyz="6.1e-05" ixz="7e-06"/>
-  </inertial>
   <visual>
     <origin xyz="0 0 0" rpy="0 0 0"/>
@@ -105,9 +80,4 @@
 </link>
 <link name="link5_1">
-  <inertial>
-    <origin xyz="-0.18454465996686803 0.41770479167069396 0.21286940543338817" rpy="0 0 0"/>
-    <mass value="0.1607410659493192"/>
-    <inertia ixx="9.1e-05" iyy="0.000104" izz="7.9e-05" ixy="-5e-06" iyz="5e-06" ixz="-8e-06"/>
-  </inertial>
   <visual>
     <origin xyz="0 0 0" rpy="0 0 0"/>
@@ -125,9 +95,4 @@
 </link>
 <link name="link6_1">
-  <inertial>
-    <origin xyz="-0.1139190355815723 0.43442970533659214 0.38100115968800496" rpy="0 0 0"/>
-    <mass value="0.01865052429923146"/>
-    <inertia ixx="1e-05" iyy="6e-06" izz="1e-05" ixy="2e-06" iyz="-1e-06" ixz="-1e-06"/>
-  </inertial>
   <visual>
     <origin xyz="0 0 0" rpy="0 0 0"/>
@@ -145,40 +110,90 @@
 </link>
 <link name="Servo_Gear_1">
-  <inertial>
-    <origin xyz="0.018998787739794347 -0.03233241707548999 0.024569258659072113" rpy="0 0 0"/>
-    <mass value="0.015458635829547249"/>
-    <inertia ixx="1.4e-05" iyy="1e-05" izz="9e-06" ixy="3e-06" iyz="6e-06" ixz="-4e-06"/>
-  </inertial>
-  <visual>
-    <origin xyz="0 0 0" rpy="0 0 0"/>
-    <geometry>
-      <mesh filename="package://robot_description/meshes/Servo_Gear_1.stl" scale="0.001 0.001 0.001"/>
-    </geometry>
-    <material name="silver"/>
-  </visual>
-  <collision>
-    <origin xyz="0 0 0" rpy="0 0 0"/>
-    <geometry>
-      <mesh filename="package://robot_description/meshes/Servo_Gear_1.stl" scale="0.001 0.001 0.001"/>
+  <visual>
+    <origin xyz="0 0 0" rpy="0 0 0"/>
+    <geometry>
+      <mesh filename="package://robot_description/meshes/Servo_Gear.stl" scale="0.001 0.001 0.001"/>
+    </geometry>
+    <material name="silver"/>
+  </visual>
+  <collision>
+    <origin xyz="0 0 0" rpy="0 0 0"/>
+    <geometry>
+      <mesh filename="package://robot_description/meshes/Servo_Gear.stl" scale="0.001 0.001 0.001"/>
+    </geometry>
+  </collision>
+</link>
+<link name="Pivot_Servo">
+  <visual>
+    <origin xyz="0 0 0" rpy="0 0 0"/>
+    <geometry>
+      <mesh filename="package://robot_description/meshes/Pivot_Arm.stl" scale="0.001 0.001 0.001"/>
+    </geometry>
+    <material name="silver"/>
+  </visual>
+  <collision>
+    <origin xyz="0 0 0" rpy="0 0 0"/>
+    <geometry>
+      <mesh filename="package://robot_description/meshes/Pivot_Arm.stl" scale="0.001 0.001 0.001"/>
+    </geometry>
+  </collision>
+</link>
+<link name="Gripper_Servo">
+  <visual>
+    <origin xyz="0 0 0" rpy="0 0 0"/>
+    <geometry>
+      <mesh filename="package://robot_description/meshes/Gripper_Servo.stl" scale="0.001 0.001 0.001"/>
+    </geometry>
+    <material name="silver"/>
+  </visual>
+  <collision>
+    <origin xyz="0 0 0" rpy="0 0 0"/>
+    <geometry>
+      <mesh filename="package://robot_description/meshes/Gripper_Servo.stl" scale="0.001 0.001 0.001"/>
     </geometry>
   </collision>
 </link>
 <link name="Idol_Gear_1">
-  <inertial>
-    <origin xyz="0.01859007116218464 0.005649685131553797 0.04057153069940722" rpy="0 0 0"/>
-    <mass value="0.01558102330322005"/>
-    <inertia ixx="1.4e-05" iyy="1.6e-05" izz="3e-06" ixy="0.0" iyz="0.0" ixz="-5e-06"/>
-  </inertial>
-  <visual>
-    <origin xyz="0 0 0" rpy="0 0 0"/>
-    <geometry>
-      <mesh filename="package://robot_description/meshes/Idol_Gear_1.stl" scale="0.001 0.001 0.001"/>
-    </geometry>
-    <material name="silver"/>
-  </visual>
-  <collision>
-    <origin xyz="0 0 0" rpy="0 0 0"/>
-    <geometry>
-      <mesh filename="package://robot_description/meshes/Idol_Gear_1.stl" scale="0.001 0.001 0.001"/>
+  <visual>
+    <origin xyz="0 0 0" rpy="0 0 0"/>
+    <geometry>
+      <mesh filename="package://robot_description/meshes/Idol_Gear.stl" scale="0.001 0.001 0.001"/>
+    </geometry>
+    <material name="silver"/>
+  </visual>
+  <collision>
+    <origin xyz="0 0 0" rpy="0 0 0"/>
+    <geometry>
+      <mesh filename="package://robot_description/meshes/Idol_Gear.stl" scale="0.001 0.001 0.001"/>
+    </geometry>
+  </collision>
+</link>
+<link name="Pivot_Idol">
+  <visual>
+    <origin xyz="0 0 0" rpy="0 0 0"/>
+    <geometry>
+      <mesh filename="package://robot_description/meshes/Pivot_Arm.stl" scale="0.001 0.001 0.001"/>
+    </geometry>
+    <material name="silver"/>
+  </visual>
+  <collision>
+    <origin xyz="0 0 0" rpy="0 0 0"/>
+    <geometry>
+      <mesh filename="package://robot_description/meshes/Pivot_Arm.stl" scale="0.001 0.001 0.001"/>
+    </geometry>
+  </collision>
+</link>
+<link name="Gripper_Idol">
+  <visual>
+    <origin xyz="0 0 0" rpy="0 0 0"/>
+    <geometry>
+      <mesh filename="package://robot_description/meshes/Gripper_Idol.stl" scale="0.001 0.001 0.001"/>
+    </geometry>
+    <material name="silver"/>
+  </visual>
+  <collision>
+    <origin xyz="0 0 0" rpy="0 0 0"/>
+    <geometry>
+      <mesh filename="package://robot_description/meshes/Gripper_Idol.stl" scale="0.001 0.001 0.001"/>
     </geometry>
   </collision>
@@ -206,5 +221,5 @@
 </joint>
 <joint name="Joint4" type="revolute">
-  <origin xyz="0 0 0.1291" rpy="0 0 0"/>
+  <origin xyz="0 0 0.1291" rpy="0 0 3.14159"/>
   <parent link="link3_1"/>
   <child link="link4_1"/>
@@ -216,5 +231,5 @@
   <parent link="link4_1"/>
   <child link="link5_1"/>
-  <axis xyz="0 1 0"/>
+  <axis xyz="0 -1 0"/>
   <limit upper="1.7" lower="-1.7" effort="100" velocity="100.0"/>
 </joint>
@@ -233,4 +248,20 @@
   <limit upper="0" lower="-1.5708" effort="100" velocity="100.0"/>
 </joint>
+<joint name="Pivot Servo Joint" type="revolute">
+  <origin xyz="0 -0.007 0.044" rpy="0 -1.5708 0"/>
+  <parent link="link6_1"/>
+  <child link="Pivot_Servo"/>
+  <mimic joint="Servo Joint"/>
+  <axis xyz="0 0 1"/>
+  <limit upper="3.14" lower="-3.14" effort="100" velocity="100.0"/>
+</joint>
+<joint name="Gripper Servo Joint" type="revolute">
+  <origin xyz="0.04 0 0" rpy="0 0 0"/>
+  <parent link="Servo_Gear_1"/>
+  <child link="Gripper_Servo"/>
+  <mimic joint="Servo Joint" multiplier="-1.0"/>
+  <axis xyz="0 0 1"/>
+  <limit upper="3.14" lower="-3.14" effort="100" velocity="100.0"/>
+</joint>
 <joint name="Idol Joint" type="revolute">
   <origin xyz="0 0.014 0.024" rpy="0 -1.5708 0"/>
@@ -241,3 +272,19 @@
   <limit upper="0" lower="-1.5708" effort="100" velocity="100.0"/>
 </joint>
+<joint name="Pivot Idol Joint" type="revolute">
+  <origin xyz="0 0.007 0.044" rpy="0 -1.5708 0"/>
+  <parent link="link6_1"/>
+  <child link="Pivot_Idol"/>
+  <mimic joint="Pivot Servo Joint"/>
+  <axis xyz="0 0 -1"/>
+  <limit upper="3.14" lower="-3.14" effort="100" velocity="100.0"/>
+</joint>
+<joint name="Gripper Idol Joint" type="revolute">
+  <origin xyz="0.04 0 0" rpy="0 0 0"/>
+  <parent link="Idol_Gear_1"/>
+  <child link="Gripper_Idol"/>
+  <mimic joint="Idol Joint" multiplier="1.0"/>
+  <axis xyz="0 0 1"/>
+  <limit upper="3.14" lower="-3.14" effort="100" velocity="100.0"/>
+</joint>
 </robot>
